File: PrototypeSingleHexTile/Untitled.kicad_pcb (KiCad board)
At the start: 2 copper layers, 44.6 x 38.6 mm, 12 parts

Commit message: v1 of the single hex (3 sizes) and single pent boards
Other:
- board text added: "Designed by Sebouh J. Paul v1 sidelength=22.30 mm"
- board text removed: "Designed by Sebouh J. Paul sidelength=22.30 mm"
Changed lines of the file:
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@@
   (gr_circle (center 93.59 40.43) (end 94.39 40.43) (layer "Edge.Cuts") (width 0.1) (fill none))
   (gr_line (start 126.04 58.01) (end 114.89 38.7) (layer "Edge.Cuts") (width 0.1))
-  (gr_text "Designed by \nSebouh J. Paul\nsidelength=22.30 mm" (at 90.8 65.4 -60) (layer "B.SilkS")
+  (gr_text "Designed by \nSebouh J. Paul\nv1\nsidelength=22.30 mm" (at 90.8 65.4 -60) (layer "B.SilkS")
     (effects (font (size 1 1) (thickness 0.15)) (justify mirror))
   )
