File: Ecal2.5x2.5cm/Ecal2.5x2.5cm.kicad_pcb (KiCad board)
At the start: 2 copper layers, 75 x 25 mm, 16 parts

Commit message: corrected capacitance in Ecal 2.5x2.5 cm^2 board
Parts:
- 10 nF: renamed from 50 nF (x4)
Changed lines of the file:
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@@
     (tags "capacitor")
     (attr smd)
-    (fp_text reference "50 nF" (at 0 -2.3 90) (layer "F.SilkS")
+    (fp_text reference "10 nF" (at 0 -2.3 90) (layer "F.SilkS")
       (effects (font (size 1 1) (thickness 0.15)))
     )
@@
     (tags "capacitor")
     (attr smd)
-    (fp_text reference "50 nF" (at 0 -2.3 90) (layer "F.SilkS")
+    (fp_text reference "10 nF" (at 0 -2.3 90) (layer "F.SilkS")
       (effects (font (size 1 1) (thickness 0.15)))
     )
@@
     (tags "capacitor")
     (attr smd)
-    (fp_text reference "50 nF" (at 0 -2.3 90) (layer "F.SilkS")
+    (fp_text reference "10 nF" (at 0 -2.3 90) (layer "F.SilkS")
       (effects (font (size 1 1) (thickness 0.15)))
     )
@@
     (tags "capacitor")
     (attr smd)
-    (fp_text reference "50 nF" (at 0 -2.3 90) (layer "F.SilkS")
-      (effects (font (size 1 1) (thickness 0.15)))
-    )
+    (fp_text reference "10 nF" (at 0 -2.3 90) (layer "F.SilkS")
+      (effects (font (size 1 1) (thickness 0.15)))
+    )
