File: Dummy Board/Dummy Board.kicad_pcb (KiCad board)
At the start: 2 copper layers, 23.6 x 7.2 mm, 1 part

Commit message: dummy board with two edgecards
Parts:
- added REF**: Samtec_HSEC8-113-X-X-DV_2x13_P0.8mm_Edge, Connector_Samtec_HSEC8:Samtec_HSEC8-113-X-X-DV_2x13_P0.8mm_Edge, B.Cu at (138.0, 73.6)
Connections:
- REF** pad 1: (no net) -> 2
- REF** pad 2: (no net) -> 1
Routing:
- net 2: track 0.00 -> 179.4 mm
- net 1: track 0.00 -> 179.4 mm
Other:
- board size 23.6 x 7.2 mm -> 23.6 x 8.6 mm
