File: PrototypeSingleHexTileLarge_6mmSiPM/Untitled.kicad_pcb (KiCad board)
At the start: 2 copper layers, 44.6 x 38.6 mm, 7 parts

Commit message: use 6050HS instead of 6015PS for single hex board
Parts:
- REF**: value S14160-3015PS -> S14160-6050HS; footprint SiPM:S14160-6010PS_dimple_silkscreen_with_LED_and_capacitor -> SiPM:S14160-6050HS_dimple_silkscreen_with_LED_and_capacitor
Other:
- board text added: "Designed by Sebouh J. Paul v4. 6 mm SiPM sidelength=22.30 mm"
- board text added: "S14160-6050HS"
- board text removed: "Designed by Sebouh J. Paul v3. 6 mm SiPM sidelength=22.30 mm"
Changed lines of the file:
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@@
 	)
 	(net 0 "")
-	(footprint "SiPM:S14160-6010PS_dimple_silkscreen_with_LED_and_capacitor"
+	(footprint "SiPM:S14160-6050HS_dimple_silkscreen_with_LED_and_capacitor"
 		(layer "F.Cu")
 		(at 103.74 58.01)
@@
 			)
 		)
-		(property "Value" "S14160-3015PS"
+		(property "Value" "S14160-6050HS"
 			(at 0 -5.8 0)
 			(unlocked yes)
@@
 			)
 		)
-		(property "Footprint" "SiPM:S14160-6010PS_dimple_silkscreen_with_LED_and_capacitor"
+		(property "Footprint" "SiPM:S14160-6050HS_dimple_silkscreen_with_LED_and_capacitor"
 			(at 0 4.9 0)
 			(unlocked yes)
@@
 		(fp_line
 			(start -4.8 -1.3)
-			(end -2.55 -2.1)
+			(end -2.5 -2.5)
 			(stroke
 				(width 0.2)
@@
 		)
 		(fp_line
-			(start -4.8 1.3)
-			(end -2.55 2.1)
+			(start -2.5 -2.5)
+			(end 2.5 -2.5)
 			(stroke
 				(width 0.2)
@@
 		)
 		(fp_line
-			(start -2.55 2.1)
-			(end -1.35 2.15)
+			(start -2.5 2.5)
+			(end 2.5 2.5)
 			(stroke
 				(width 0.2)
@@
 		)
 		(fp_line
-			(start -1.35 2.15)
-			(end 0.775 4.25)
+			(start -1.25 -1.25)
+			(end 1.25 -1.25)
 			(stroke
 				(width 0.2)
@@
 		)
 		(fp_line
+			(start -1.25 1.25)
+			(end -4.8 1.3)
+			(stroke
+				(width 0.2)
+				(type default)
+			)
+			(layer "F.Cu")
+		)
+		(fp_line
 			(start -0.775 4.25)
 			(end -2.575 4.725)
@@
 		)
 		(fp_line
-			(start -0.775 4.25)
-			(end -0.7 5.3)
+			(start -0.65 2.5)
+			(end 0.775 4.25)
 			(stroke
 				(width 0.2)
@@
 		)
 		(fp_line
-			(start -0.7 5.3)
-			(end 2 5.3)
+			(start 0.875 -4.285)
+			(end 2 -4.3)
 			(stroke
 				(width 0.2)
@@
 		)
 		(fp_line
-			(start 0.875 -4.285)
-			(end 2 -4.3)
+			(start 1.25 -1.25)
+			(end 1.25 1.25)
 			(stroke
 				(width 0.2)
@@
 		)
 		(fp_line
-			(start 1.9 3.3)
-			(end 0 1.3)
+			(start 1.25 1.25)
+			(end -1.25 1.25)
 			(stroke
 				(width 0.2)
@@
 		)
 		(fp_line
-			(start 2 5.3)
-			(end 1.9 3.3)
+			(start 2.5 -2.5)
+			(end 2.5 2.5)
 			(stroke
 				(width 0.2)
@@
 		)
 		(fp_line
-			(start -7.675 0.25)
-			(end -6.375 0.25)
-			(stroke
-				(width 0.12)
-				(type solid)
-			)
-			(layer "F.SilkS")
-		)
-		(fp_line
-			(start -7.075 1.35)
-			(end -7.075 -1.65)
+			(start 2.5 2.5)
+			(end 2.5 -2.5)
+			(stroke
+				(width 0.2)
+				(type default)
+			)
+			(layer "F.Cu")
+		)
+		(fp_line
+			(start -7.675 -0.55)
+			(end -6.375 -0.55)
+			(stroke
+				(width 0.12)
+				(type solid)
+			)
+			(layer "F.SilkS")
+		)
+		(fp_line
+			(start -7.075 -1.65)
+			(end -7.075 1.35)
 			(stroke
 				(width 0.12)
@@
 		)
 		(fp_line
-			(start -3.925 3.425)
-			(end 3.425 3.425)
+			(start -3.2 -3.2)
+			(end -3.2 3.2)
+			(stroke
+				(width 0.12)
+				(type default)
+			)
+			(layer "F.SilkS")
+		)
+		(fp_line
+			(start -3.2 3.2)
+			(end 3.2 3.2)
 			(stroke
 				(width 0.12)
@@
 		)
 		(fp_line
-			(start 3.425 -3.425)
-			(end -3.925 -3.425)
-			(stroke
-				(width 0.12)
-				(type solid)
-			)
-			(layer "F.SilkS")
-		)
-		(fp_line
-			(start 3.425 -3.425)
-			(end 3.425 3.425)
-			(stroke
-				(width 0.12)
-				(type solid)
-			)
+			(start 3.2 -3.2)
+			(end -3.2 -3.2)
+			(stroke
+				(width 0.12)
+				(type default)
+			)
+			(layer "F.SilkS")
+		)
+		(fp_line
+			(start 3.2 3.2)
+			(end 3.2 -3.2)
+			(stroke
+				(width 0.12)
+				(type default)
+			)
+			(layer "F.SilkS")
+		)
+		(fp_rect
+			(start -3.3 -3.45)
+			(end 3.2 -3.2)
+			(stroke
+				(width 0.12)
+				(type solid)
+			)
+			(fill solid)
 			(layer "F.SilkS")
 		)
@@
 		)
 		(fp_rect
+			(start -1.6 3.2)
+			(end 1.55 3.45)
+			(stroke
+				(width 0.12)
+				(type solid)
+			)
+			(fill solid)
+			(layer "F.SilkS")
+		)
+		(fp_rect
+			(start 3.2 -3.45)
+			(end 3.45 3.2)
+			(stroke
+				(width 0.12)
+				(type solid)
+			)
+			(fill solid)
+			(layer "F.SilkS")
+		)
+		(fp_rect
 			(start 4.6 -0.625)
 			(end 3.375 -1.4)
@@
 		(fp_poly
 			(pts
-				(xy -7.075 0.25) (xy -7.675 -0.75) (xy -6.475 -0.75)
+				(xy -7.075 -0.55) (xy -7.675 0.45) (xy -6.475 0.45)
 			)
 			(stroke
@@
 		(fp_poly
 			(pts
-				(xy 1.55 3.45) (xy 1.55 5.7) (xy 2.15 5.55) (xy 2.95 5.15) (xy 3.55 4.75) (xy 4.1 4.3) (xy 4.75 3.55)
-				(xy 4.65 2.6) (xy 3.5 2.6) (xy 3.5 3.5)
+				(xy 1.55 3.2) (xy 1.55 5.7) (xy 2.15 5.55) (xy 2.95 5.15) (xy 3.55 4.75) (xy 4.1 4.3) (xy 4.75 3.55)
+				(xy 4.65 2.6) (xy 3.5 2.6) (xy 3.2 3.2)
 			)
 			(stroke
@@
 			(pts
 				(xy -4 4.35) (xy -4.65 3.65) (xy -5.35 2.6) (xy -5.85 1.05) (xy -5.95 0) (xy -5.85 -1.05) (xy -5.5 -2.3)
-				(xy -4.95 -3.35) (xy -4.3 -4.1) (xy -3.95 -3.4) (xy -3.95 3.5)
+				(xy -4.95 -3.35) (xy -4.3 -4.1) (xy -3.2 -3.2) (xy -3.2 3.2)
 			)
 			(stroke
@@
 		(fp_poly
 			(pts
-				(xy 1.55 5.05) (xy -1.55 5.05) (xy -1.55 3.45) (xy -3.925 3.425) (xy -3.95 4.5) (xy -2.85 5.25)
-				(xy -1.7 5.7) (xy -0.6 5.9) (xy 0.55 5.9) (xy 1 5.85) (xy 1.6 5.75)
+				(xy 1.55 5.05) (xy -1.55 5.05) (xy -1.55 3.2) (xy -3.9 3.2) (xy -3.95 4.5) (xy -2.85 5.25) (xy -1.7 5.7)
+				(xy -0.6 5.9) (xy 0.55 5.9) (xy 1 5.85) (xy 1.6 5.75)
 			)
 			(stroke
@@
 		(fp_poly
 			(pts
-				(xy 3.4 -3.55) (xy 3.35 -4.85) (xy 4.25 -4.15) (xy 4.95 -3.25) (xy 5.3 -2.65) (xy 5.65 -1.85) (xy 5.85 -1)
+				(xy 3.2 -3.55) (xy 3.35 -4.85) (xy 4.25 -4.15) (xy 4.95 -3.25) (xy 5.3 -2.65) (xy 5.65 -1.85) (xy 5.85 -1)
 				(xy 5.95 -0.05) (xy 5.85 1.05) (xy 5.5 2.25) (xy 4.9 3.35) (xy 4.75 3.55) (xy 4.65 2.6) (xy 4.6 -2.6)
-				(xy 3.4 -2.6)
+				(xy 3.2 -2.6)
 			)
 			(stroke
@@
 		)
 		(fp_text user "${REFERENCE}"
+			(at 0 -4.3 0)
+			(layer "F.Fab")
+			(effects
+				(font
+					(size 0.4 0.4)
+					(thickness 0.06)
+				)
+			)
+		)
+		(fp_text user "${REFERENCE}"
 			(at 0 -6.8 0)
 			(unlocked yes)
@@
 			)
 		)
-		(fp_text user "${REFERENCE}"
-			(at 0 -4.3 0)
-			(layer "F.Fab")
-			(effects
-				(font
-					(size 0.4 0.4)
-					(thickness 0.06)
-				)
-			)
-		)
 		(pad "1" smd circle
-			(at -2.55 2.1)
-			(size 1.1 1.1)
+			(at -2.5 2.5)
+			(size 0.7 0.7)
+			(layers "F.Cu" "F.Paste" "F.Mask")
+		)
+		(pad "1" smd circle
+			(at -1.25 1.25)
+			(size 0.7 0.7)
 			(layers "F.Cu" "F.Paste" "F.Mask")
 		)
@@
 		)
 		(pad "2" smd circle
-			(at 2.05 2.1)
-			(size 1.1 1.1)
+			(at 1.25 1.25)
+			(size 0.7 0.7)
 			(layers "F.Cu" "F.Paste" "F.Mask")
 		)
+		(pad "2" smd circle
+			(at 2.5 2.5)
+			(size 0.7 0.7)
+			(layers "F.Cu" "F.Paste" "F.Mask")
+		)
 		(pad "3" smd circle
-			(at -2.55 -2.1)
-			(size 1.1 1.1)
+			(at -2.5 -2.5)
+			(size 0.7 0.7)
 			(layers "F.Cu" "F.Paste" "F.Mask")
 		)
+		(pad "3" smd circle
+			(at -1.25 -1.25)
+			(size 0.7 0.7)
+			(layers "F.Cu" "F.Paste" "F.Mask")
+		)
 		(pad "4" smd circle
-			(at 2.05 -2.1)
-			(size 1.1 1.1)
+			(at 1.25 -1.25)
+			(size 0.7 0.7)
+			(layers "F.Cu" "F.Paste" "F.Mask")
+		)
+		(pad "4" smd circle
+			(at 2.5 -2.5)
+			(size 0.7 0.7)
 			(layers "F.Cu" "F.Paste" "F.Mask")
 		)
@@
 			(remove_unused_layers no)
 		)
-		(pad "10" smd rect
-			(at -0.25 0 45)
-			(size 3.5 3.5)
-			(layers "F.Cu" "F.Paste" "F.Mask")
-			(thermal_bridge_angle 45)
-		)
 	)
 	(footprint "Sensor:LM94021QBIMG-NOPB"
@@
 		(at 103.7 58 180)
 		(property "Reference" "REF**"
-			(at 0 0.5 0)
+			(at 0.7 -3.2 0)
 			(unlocked yes)
 			(layer "B.SilkS")
@@
 		(layer "Edge.Cuts")
 	)
-	(gr_text "Designed by \nSebouh J. Paul\nv3.  6 mm SiPM\nsidelength=22.30 mm"
+	(gr_text "Designed by \nSebouh J. Paul\nv4.  6 mm SiPM\nsidelength=22.30 mm"
 		(at 90.8 65.4 300)
 		(layer "B.SilkS")
@@
 		)
 	)
+	(gr_text "S14160-6050HS"
+		(at 97.6 48.6 0)
+		(layer "F.SilkS")
+		(effects
+			(font
+				(size 1 1)
+				(thickness 0.15)
+			)
+			(justify left bottom)
+		)
+	)
