File: ZDC_Prototype/EvenLayers_1.3mm_SiPM/EvenLayers_1.3mm_SiPM.kicad_pcb (KiCad board)
At the start: 2 copper layers, 295 x 300 mm, 37 parts

Commit message: updated 1.3 mm boards
Parts:
- moved G*** 5.00 mm to (302.5, 41.9)
- moved G*** 5.00 mm to (273.6, 55.1)
- moved G*** 5.00 mm to (232.5, 53.3)
- moved G*** 5.00 mm to (308.2, 62.4)
- moved REF**44 3.18 mm to (324.8, 289.8)
- moved REF**24 2.85 mm to (324.8, 94.6)
- moved REF**40 2.85 mm to (129.6, 289.8)
- moved REF**39 2.57 mm to (324.8, 241.0)
- moved REF**43 2.57 mm to (276.0, 289.8)
- moved REF**20 2.47 mm to (129.6, 94.6)
- moved REF**29 2.37 mm to (324.8, 143.4)
- moved REF**41 2.37 mm to (178.4, 289.8)
- moved REF**34 2.26 mm to (324.8, 192.2)
- moved REF**42 2.26 mm to (227.2, 289.8)
- moved REF**23 2.15 mm to (276.0, 94.6)
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Routing:
- net GND: track 1944.6 -> 1830.3 mm
- net A6: track 132.3 -> 124.3 mm
- net K5: track 75.0 -> 67.1 mm
- net K6: track 126.7 -> 119.1 mm
- net (no net): track 2139.8 -> 2132.3 mm
- net K10: track 92.0 -> 85.1 mm
- net K15: track 82.3 -> 75.4 mm
- net A5: track 80.0 -> 73.5 mm
- net A10: track 97.4 -> 91.1 mm
- net A15: track 87.3 -> 81.6 mm
- net A16: track 141.1 -> 135.6 mm
- net K16: track 135.4 -> 130.1 mm
- net A11: track 150.8 -> 146.0 mm
- net K21: track 158.5 -> 154.3 mm
- net K11: track 145.1 -> 140.9 mm
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Other:
- board size 295 x 300 mm -> 297 x 290 mm
- board text added: "SiPM size: 1.3 mm space between SiPMs: 48.8 mm Absorber area: ~30x30 cm (3x3 blocks)"
- board text added: "SiPM size: 1.3 mm space between SiPMs: 48.8 mm Absorber area: ~30x30 cm (3x3 blocks) Hole positions (relative to UL corner, mm): (15, 25) (15, 145) (15, 265) Hole radii are all 1.6 mm"
- board text added: "active area to edge 2.8 mm"
- board text removed: "3.55 mm from active area to edge"
- board text removed: "SiPM size: 1.3 mm space between SiPMs: 47.8 mm Absorber area: ~30x30 cm (3x3 blocks)"
- board text removed: "SiPM size: 1.3 mm space between SiPMs: 47.8 mm Absorber area: ~30x30 cm (3x3 blocks) Hole positions (relative to UL corner, mm): (15, 30) (15, 150) (15, 270) Hole radii are all 1.6 mm"

Commit message: version 5 of the 1.3 mm boards for the ZDC prototype
Connections:
- 50 Ω pad 1: (no net) -> LED_input
- 50 Ω pad 2: (no net) -> LED_input_after_resistor
- LEDs pad 1: (no net) -> LED_input
- REF**43 pad 6: (no net) -> LED_23_to_24
- REF**44 pad 5: (no net) -> LED_23_to_24
- REF**44 pad 6: (no net) -> LED_input_after_resistor
Routing:
- net (no net): track 2132.3 -> 1833.3 mm, vias 1 -> 0
- net LED_input_after_resistor: track 0.00 -> 287.2 mm, vias 0 -> 1
- net LED_23_to_24: track 0.00 -> 44.8 mm
- net GND: track 1830.3 -> 1785.6 mm
- net LED_input: track 0.00 -> 11.6 mm
- net A9: track 277.8 -> 280.3 mm
- net A14: track 274.0 -> 276.4 mm
- net K14: track 268.9 -> 271.3 mm
- net K9: track 272.9 -> 275.0 mm
- added copper zone on In1.Cu, net GND
Other:
- copper layers 2 -> 4
- board text added: "Designed by Sebouh J Paul Version 5 Even layers 1.3 mm SiPMs"
- board text removed: "Designed by Sebouh J Paul Version 4 Even layers 1.3 mm SiPMs"
