File: ZDC_Prototype/EvenLayers_1.3mm_SiPM/EvenLayers_1.3mm_SiPM.kicad_pcb (KiCad board)
At the start: 4 copper layers, 297 x 290 mm, 37 parts

Commit message: v8 of ZDC boards
Routing:
- net A24: track 313.9 -> 307.8 mm
- net K24: track 307.9 -> 303.6 mm
- net A12: track 203.9 -> 199.8 mm
- net A23: track 261.2 -> 257.8 mm
- net A22: track 211.6 -> 208.5 mm
- net K23: track 256.3 -> 253.2 mm
- net K22: track 206.6 -> 203.9 mm
- net A19: track 288.2 -> 286.9 mm
- net K19: track 282.7 -> 281.6 mm
- net K8: track 224.8 -> 225.6 mm
- net K2: track 180.5 -> 179.8 mm
- net A4: track 283.0 -> 283.6 mm
- added copper zone on B.Cu, net GND
- added copper zone on F.Cu, net GND
- removed copper zone on In1.Cu, net GND
Other:
- copper layers 4 -> 2
- board text added: "Designed by Sebouh J Paul Version 8 Even layers 1.3 mm SiPMs"
- board text removed: "Designed by Sebouh J Paul Version 7 Even layers 1.3 mm SiPMs"

Commit message: fixed version of even layers s v8
Connections:
- REF** pad 25: GND -> A25
- REF** pad 26: GND -> K25
Routing:
- net GND: track 1794.4 -> 1786.1 mm
Changed lines of the file:
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@@
 	(net 53 "LED_input_after_resistor")
 	(net 54 "LED_23_to_24")
+	(net 55 "A25")
+	(net 56 "K25")
 	(footprint "SiPM:S14160-1315PS_dimple_silkscreen_with_LED_and_capacitor"
 		(layer "F.Cu")
@@
 			(size 0.5 1.2)
 			(layers "F.Cu" "F.Paste" "F.Mask")
-			(net 1 "GND")
+			(net 55 "A25")
 			(solder_mask_margin 0.102)
 		)
@@
 			(size 0.5 1.2)
 			(layers "F.Cu" "F.Paste" "F.Mask")
-			(net 1 "GND")
+			(net 56 "K25")
 			(solder_mask_margin 0.102)
 		)
@@
 		)
 		(height -12.4)
-		(gr_text "35.2 mm"
+		(gr_text "1.4 in"
 			(at 332.891574 51.801574 90)
 			(layer "F.SilkS")
@@
 		)
 		(height 0)
-		(gr_text "290.0 mm"
+		(gr_text "11.4 in"
 			(at 345.4 181.4 90)
 			(layer "F.SilkS")
@@
 		)
 		(height -0.01)
-		(gr_text "297.0 mm"
+		(gr_text "11.7 in"
 			(at 197.3 318.9 359.961417)
 			(layer "F.SilkS")
@@
 		)
 		(height 1.937173)
-		(gr_text "288.0 mm"
+		(gr_text "11.3 in"
 			(at 222 272 0)
 			(layer "F.SilkS")
@@
 		)
 		(height -101.52)
-		(gr_text "244.0 mm"
+		(gr_text "9.6 in"
 			(at 246.055002 192.220567 -89.98825906)
 			(layer "F.SilkS")
@@
 		)
 		(height 5.246903)
-		(gr_text "10.8 mm"
+		(gr_text "0.4 in"
 			(at 339 320.2 90)
 			(layer "F.SilkS")
@@
 		)
 		(height -60.97)
-		(gr_text "244.0 mm"
+		(gr_text "9.6 in"
 			(at 227.2 249.33 0)
 			(layer "F.SilkS")
@@
 		)
 		(height -2.580771)
-		(gr_text "41.20 mm"
+		(gr_text "1.62 in"
 			(at 91.11 294.670771 0)
 			(layer "F.SilkS")
@@
 	)
 	(segment
-		(start 65.2 229.9)
-		(end 61.7 226.4)
-		(width 0.2)
-		(layer "F.Cu")
-		(net 1)
-	)
-	(segment
 		(start 56.6 313.4)
 		(end 59 311)
@@
 		(layer "F.Cu")
 		(net 1)
-	)
-	(segment
-		(start 58.3 226.4)
-		(end 61.7 226.4)
-		(width 0.2)
-		(layer "F.Cu")
-		(net 1)
