File: ZDC_Prototype/OddLayers_1.3mm_SiPM/OddLayers_1.3mm_SiPM.kicad_pcb (KiCad board)
At the start: 2 copper layers, 295 x 300 mm, 37 parts

Commit message: updated odd layers 1.3 mm:  correct size for the PCB board and tiles
Parts:
- moved REF**20 3.18 mm to (105.2, 70.2)
- moved REF**24 2.85 mm to (300.4, 70.2)
- moved REF**40 2.85 mm to (105.2, 265.4)
- moved REF**21 2.57 mm to (154.0, 70.2)
- moved REF**25 2.57 mm to (105.2, 119.0)
- moved REF**44 2.47 mm to (300.4, 265.4)
- moved REF**23 2.37 mm to (251.6, 70.2)
- moved REF**35 2.37 mm to (105.2, 216.6)
- moved REF**22 2.26 mm to (202.8, 70.2)
- moved REF**30 2.26 mm to (105.2, 167.8)
- moved REF**29 2.15 mm to (300.4, 119.0)
- moved REF**41 2.15 mm to (154.0, 265.4)
- moved REF**39 1.90 mm to (300.4, 216.6)
- moved REF**43 1.90 mm to (251.6, 265.4)
- moved REF**26 1.77 mm to (154.0, 119.0)
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Routing:
- net GND: track 1980.7 -> 1807.9 mm
- net (no net): track 2125.3 -> 2160.5 mm
- net K16: track 135.7 -> 125.2 mm
- net K21: track 150.3 -> 159.1 mm
- net A24: track 320.1 -> 312.4 mm
- net A0: track 61.7 -> 55.6 mm
- net K0: track 56.9 -> 51.2 mm
- net A23: track 259.6 -> 262.6 mm
- net K4: track 244.5 -> 247.5 mm
- net A4: track 250.0 -> 253.0 mm
- net K24: track 305.8 -> 308.8 mm
- net K3: track 196.6 -> 199.1 mm
- net K1: track 100.1 -> 102.5 mm
- net A3: track 201.6 -> 203.9 mm
- net K8: track 207.1 -> 209.4 mm
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Other:
- board size 295 x 300 mm -> 297 x 290 mm
- board text added: "SiPM size: 1.3 mm space between SiPMs: 48.8 mm Absorber area: ~30x30 cm (3x3 blocks)"
- board text added: "SiPM size: 1.3 mm space between SiPMs: 48.8 mm Absorber area: ~30x30 cm (3x3 blocks) Hole positions (relative to UL corner, mm): (15, 25) (15, 145) (15, 265) Hole radii are all 1.6 mm"
- board text removed: "SiPM size: 1.3 mm space between SiPMs: 47.8 mm Absorber area: ~30x30 cm (3x3 blocks)"
- board text removed: "SiPM size: 1.3 mm space between SiPMs: 47.8 mm Absorber area: ~30x30 cm (3x3 blocks) Hole positions (relative to UL corner, mm): (15, 30) (15, 150) (15, 270) Hole radii are all 1.6 mm"

Commit message: version 5 of the 1.3 mm boards for the ZDC prototype
Connections:
- 50 Ω pad 1: (no net) -> LED_input
- 50 Ω pad 2: (no net) -> LED_input_after_resistor
- LEDs pad 1: (no net) -> LED_input
- REF**44 pad 6: (no net) -> LED_input_after_resistor
Routing:
- net (no net): track 2160.5 -> 1880.6 mm, vias 1 -> 0
- net LED_input_after_resistor: track 0.00 -> 268.3 mm, vias 0 -> 1
- net LED_input: track 0.00 -> 11.6 mm
- added copper zone on In1.Cu, net GND
Other:
- copper layers 2 -> 4
- board text added: "Designed by Sebouh J Paul Version 5 Odd layers 1.3 mm SiPMs"
- board text removed: "Designed by Sebouh J Paul Version 4 Odd layers 1.3 mm SiPMs"
