File: ZDC_Prototype/OddLayers_1.3mm_SiPM/OddLayers_1.3mm_SiPM.kicad_pcb (KiCad board)
At the start: 4 copper layers, 297 x 290 mm, 37 parts

Commit message: v8 of ZDC boards
Routing:
- net LED_input_after_resistor: track 256.4 -> 276.4 mm
- net A15: track 80.5 -> 68.0 mm
- net K15: track 73.1 -> 62.6 mm
- net K14: track 251.9 -> 248.3 mm
- net A19: track 275.7 -> 272.6 mm
- net K19: track 270.9 -> 268.3 mm
- net A12: track 199.4 -> 201.9 mm
- net A11: track 150.8 -> 153.3 mm
- net A18: track 228.4 -> 226.0 mm
- net A20: track 107.6 -> 106.1 mm
- net K20: track 100.9 -> 99.5 mm
- net A13: track 205.2 -> 204.0 mm
- net A24: track 312.4 -> 311.3 mm
- net K24: track 308.8 -> 307.7 mm
- net A23: track 262.7 -> 263.6 mm
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- added copper zone on B.Cu, net GND
- added copper zone on F.Cu, net GND
- removed copper zone on In1.Cu, net GND
Other:
- copper layers 4 -> 2
- board text added: "Designed by Sebouh J Paul Version 8 Odd layers 1.3 mm SiPMs"
- board text removed: "Designed by Sebouh J Paul Version 7 Odd layers 1.3 mm SiPMs"
