File: ZDC_Prototype/OddLayers_1.3mm_SiPM/OddLayers_1.3mm_SiPM.kicad_pcb (KiCad board)
At the start: 2 copper layers, 297 x 290 mm, 37 parts

Commit message: fixed version of odd layers v8
Connections:
- REF** pad 25: GND -> A25
- REF** pad 26: GND -> K25
Routing:
- net GND: track 1769.5 -> 1645.1 mm
Changed lines of the file:
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@@
 	(net 52 "LED_input")
 	(net 53 "LED_input_after_resistor")
+	(net 54 "A25")
+	(net 55 "K25")
 	(footprint "SiPM:S14160-1315PS_dimple_silkscreen_with_LED_and_capacitor"
 		(layer "F.Cu")
@@
 			(size 0.5 1.2)
 			(layers "F.Cu" "F.Paste" "F.Mask")
-			(net 1 "GND")
+			(net 54 "A25")
 			(solder_mask_margin 0.102)
 		)
@@
 			(size 0.5 1.2)
 			(layers "F.Cu" "F.Paste" "F.Mask")
-			(net 1 "GND")
+			(net 55 "K25")
 			(solder_mask_margin 0.102)
 		)
@@
 		)
 		(height 0)
-		(gr_text "290.0 mm"
+		(gr_text "11.4 in"
 			(at 346 181.1 -89.96048568)
 			(layer "F.SilkS")
@@
 		)
 		(height 2.44133)
-		(gr_text "27.2 mm"
+		(gr_text "1.1 in"
 			(at 335.9 197.5 0)
 			(layer "F.SilkS")
@@
 		)
 		(height 5.342349)
-		(gr_text "35.2 mm"
+		(gr_text "1.4 in"
 			(at 148 310 90)
 			(layer "F.SilkS")
@@
 		)
 		(height 1.937173)
-		(gr_text "288.00 mm"
+		(gr_text "11.34 in"
 			(at 203 250 0)
 			(layer "F.SilkS")
@@
 		)
 		(height -2.624329)
-		(gr_text "10.8 mm"
+		(gr_text "0.4 in"
 			(at 292.7 41 -89.87092556)
 			(layer "F.SilkS")
@@
 		)
 		(height -0.01)
-		(gr_text "297.0 mm"
+		(gr_text "11.7 in"
 			(at 196.8 293.5 0)
 			(layer "F.SilkS")
@@
 		)
 		(height -101.52)
-		(gr_text "244.0 mm"
+		(gr_text "9.6 in"
 			(at 222.13 167.8 90)
 			(layer "F.SilkS")
@@
 		)
 		(height 2.000024)
-		(gr_text "16.8 mm"
+		(gr_text "0.7 in"
 			(at 72.11087 257.089106 0)
 			(layer "F.SilkS")
@@
 		)
 		(height -60.97)
-		(gr_text "244.0 mm"
+		(gr_text "9.6 in"
 			(at 202.8 227.68 0)
 			(layer "F.SilkS")
@@
 	)
 	(segment
-		(start 68.9 286)
-		(end 58 286)
-		(width 0.2)
-		(layer "F.Cu")
-		(net 1)
-	)
-	(segment
 		(start 56.46 297.54)
 		(end 61.54 297.54)
@@
 	)
 	(segment
-		(start 65.2 189.2)
-		(end 65.2 192.697058)
-		(width 0.2)
-		(layer "F.Cu")
-		(net 1)
-	)
-	(segment
-		(start 65.2 192.697058)
-		(end 68.9 196.397058)
-		(width 0.2)
-		(layer "F.Cu")
-		(net 1)
-	)
-	(segment
-		(start 61.7 186.4)
-		(end 62.4 186.4)
-		(width 0.2)
-		(layer "F.Cu")
-		(net 1)
-	)
-	(segment
 		(start 76 300)
 		(end 74.975 301.025)
@@
 	)
 	(segment
-		(start 58 286)
-		(end 56.46 287.54)
-		(width 0.2)
-		(layer "F.Cu")
-		(net 1)
-	)
-	(segment
 		(start 56.46 297.54)
 		(end 56.46 292.46)
 		(width 0.2)
 		(layer "F.Cu")
-		(net 1)
-	)
-	(segment
-		(start 58.3 186.4)
-		(end 61.7 186.4)
-		(width 0.2)
-		(layer "F.Cu")
-		(net 1)
-	)
-	(segment
-		(start 62.4 186.4)
-		(end 65.2 189.2)
-		(width 0.2)
-		(layer "F.Cu")
-		(net 1)
-	)
-	(segment
-		(start 56.46 287.54)
-		(end 56.46 292.46)
-		(width 0.2)
-		(layer "F.Cu")
-		(net 1)
-	)
-	(segment
-		(start 68.9 196.397058)
-		(end 68.9 286)
-		(width 0.2)
-		(layer "F.Cu")
