File: OctagonPanels/OctagonPanels.kicad_pcb (KiCad board)
At the start: 4 copper layers, 420.4 x 48.8 mm, 13 parts

Commit message: updated documentation on board
Other:
- board text added: "Designed by Sebouh J Paul 1.3 mm SiPMs 48.8 x 48.8 mm2 scint cells connectors: SAMTEC_HSEC8-113-01-X-DV-A-L2 JST B3B-XH-A temp sensor: LM94021QBIMGX/NOPB capacitors: AGC0603X7R101-103KNP Version 1"
Changed lines of the file:
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@@
 		)
 		(property "Value" "SAMTEC_HSEC8-113-01-X-DV-A-L2"
-			(at 6.985 -8.255 90)
+			(at 0 -8.255 90)
 			(layer "B.Fab")
 			(effects
@@
 		)
 	)
-	(gr_text "Designed by \nSebouh J Paul\n\n1.3 mm SiPMs\n48.8 x 48.8 mm2 scint cells\nVersion 1"
-		(at 182.7 95.2 0)
+	(gr_text "Designed by \nSebouh J Paul\n\n1.3 mm SiPMs\n48.8 x 48.8 mm2 scint cells\nconnectors:\nSAMTEC_HSEC8-113-01-X-DV-A-L2 \nJST B3B-XH-A\ntemp sensor:\nLM94021QBIMGX/NOPB\ncapacitors:\nAGC0603X7R101-103KNP\nVersion 1"
+		(at 134.9 83.65 0)
 		(layer "B.SilkS")
 		(effects
@@
 		)
 	)
+	(gr_text "Designed by \nSebouh J Paul\n\n1.3 mm SiPMs\n48.8 x 48.8 mm2 scint cells\nVersion 1"
+		(at 182.7 95.2 -0)
+		(layer "F.SilkS")
+		(effects
+			(font
+				(size 1.5 1.5)
+				(thickness 0.3)
+			)
+		)
+	)
 	(gr_text "1"
 		(at 85.85 72.8 0)
@@
 			)
 		)
-	)
-	(gr_text "Designed by \nSebouh J Paul\n\n1.3 mm SiPMs\n48.8 x 48.8 mm2 scint cells\nVersion 1"
-		(at 131.1 95.4 0)
-		(layer "F.SilkS")
-		(effects
-			(font
-				(size 1.5 1.5)
-				(thickness 0.3)
-			)
-		)
